File: Token_Ring_MAU.kicad_pcb (KiCad board)
At the start: 4 copper layers, 100 x 70 mm, 62 parts, among them J1 RJ45_LED_Shielded_x2, J200 Barrel_Jack, J201 12V Jumper, J202 5V Jumper, K1 4PDT_relay, K2 4PDT_relay, Q1 Q_NPN_BEC, Q2 Q_NPN_BEC, Q21 Q_NPN_BEC, Q22 Q_NPN_BEC, T1 Transformer_Token_Ring_1to1_1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, T2 Transformer_Token_Ring_1to1_1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, U1 H11A1, U200 KA78M05_TO252, U21 H11A1

Commit message: Add pictures, gerbers, warning note
Parts:
- C200: footprint Capacitor_SMD:CP_Elec_5x5.9 -> Capacitor_SMD:CP_Elec_5x5.8
- C201, C202: value 0.1uF -> 100n
- D1, D21: footprint Diode_SMD:D_0805_2012Metric_Pad1.15x1.40mm_HandSolder -> Diode_SMD:D_SOD-123F
