File: Token_Ring_MAU.kicad_sch (KiCad schematic)
At the start: 11 parts, among them J200 Barrel_Jack, J201 12V Jumper, J202 5V Jumper, U200 KA78M05_TO252

Commit message: Add pictures, gerbers, warning note
Parts:
- C200: value 0.33u -> 33u; footprint Capacitor_SMD:CP_Elec_5x5.9 -> Capacitor_SMD:CP_Elec_5x5.8; JLCPCB part number (none) -> C128455; LCSC (none) -> C128455
- C201, C202: value 0.1uF -> 100n; JLCPCB part number (none) -> C85866; LCSC (none) -> C85866
- H1, H2, H3, H4, J200, J201, J202, U200: JLCPCB part number (none) -> DNP; LCSC (none) -> DNP
Changed lines of the file:
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@@
+      (effects (font (size 1.27 1.27)) hide)
+    )
+    (property "JLCPCB part number" "DNP" (id 4) (at 241.935 81.28 0)
+      (effects (font (size 1.27 1.27)) hide)
+    )
+    (property "LCSC" "DNP" (id 5) (at 241.935 81.28 0)
       (effects (font (size 1.27 1.27)) hide)
     )
@@
       (effects (font (size 1.27 1.27)) hide)
     )
+    (property "JLCPCB part number" "DNP" (id 4) (at 207.01 81.28 0)
+      (effects (font (size 1.27 1.27)) hide)
+    )
+    (property "LCSC" "DNP" (id 5) (at 207.01 81.28 0)
+      (effects (font (size 1.27 1.27)) hide)
+    )
     (pin "1")
     (pin "2")
@@
       (effects (font (size 1.27 1.27)) (justify left))
     )
-    (property "Value" "0.33u" (id 1) (at 175.895 85.725 0)
-      (effects (font (size 1.27 1.27)) (justify left))
-    )
-    (property "Footprint" "Capacitor_SMD:CP_Elec_5x5.9" (id 2) (at 186.3852 88.9 0)
+    (property "Value" "33u" (id 1) (at 175.895 85.725 0)
+      (effects (font (size 1.27 1.27)) (justify left))
+    )
+    (property "Footprint" "Capacitor_SMD:CP_Elec_5x5.8" (id 2) (at 186.3852 88.9 0)
       (effects (font (size 1.27 1.27)) hide)
     )
     (property "Datasheet" "~" (id 3) (at 185.42 85.09 0)
+      (effects (font (size 1.27 1.27)) hide)
+    )
+    (property "JLCPCB part number" "C128455" (id 4) (at 185.42 85.09 0)
+      (effects (font (size 1.27 1.27)) hide)
+    )
+    (property "LCSC" "C128455" (id 5) (at 185.42 85.09 0)
       (effects (font (size 1.27 1.27)) hide)
     )
@@
       (effects (font (size 1.27 1.27)) hide)
     )
+    (property "JLCPCB part number" "DNP" (id 4) (at 207.645 60.96 0)
+      (effects (font (size 1.27 1.27)) hide)
+    )
+    (property "LCSC" "DNP" (id 5) (at 207.645 60.96 0)
+      (effects (font (size 1.27 1.27)) hide)
+    )
     (pin "1")
     (pin "2")
@@
       (effects (font (size 1.27 1.27)) hide)
     )
+    (property "JLCPCB part number" "DNP" (id 4) (at 220.345 59.69 0)
+      (effects (font (size 1.27 1.27)) hide)
+    )
+    (property "LCSC" "DNP" (id 5) (at 220.345 59.69 0)
+      (effects (font (size 1.27 1.27)) hide)
+    )
     (pin "1")
     (pin "2")
@@
       (effects (font (size 1.27 1.27)) hide)
     )
+    (property "JLCPCB part number" "DNP" (id 4) (at 210.185 42.545 0)
+      (effects (font (size 1.27 1.27)) hide)
+    )
+    (property "LCSC" "DNP" (id 5) (at 210.185 42.545 0)
+      (effects (font (size 1.27 1.27)) hide)
+    )
   )
   (symbol (lib_id "Mechanical:MountingHole") (at 210.185 36.195 0) (unit 1)
@@
     )
     (property "Datasheet" "~" (id 3) (at 210.185 36.195 0)
+      (effects (font (size 1.27 1.27)) hide)
+    )
+    (property "JLCPCB part number" "DNP" (id 4) (at 210.185 36.195 0)
+      (effects (font (size 1.27 1.27)) hide)
+    )
+    (property "LCSC" "DNP" (id 5) (at 210.185 36.195 0)
       (effects (font (size 1.27 1.27)) hide)
     )
@@
       (effects (font (size 1.27 1.27)) hide)
     )
+    (property "JLCPCB part number" "DNP" (id 4) (at 210.185 29.845 0)
+      (effects (font (size 1.27 1.27)) hide)
+    )
+    (property "LCSC" "DNP" (id 5) (at 210.185 29.845 0)
+      (effects (font (size 1.27 1.27)) hide)
+    )
   )
   (symbol (lib_id "power:+12V") (at 215.9 140.97 0) (unit 1)
@@
     )
     (property "Datasheet" "~" (id 3) (at 210.185 23.495 0)
+      (effects (font (size 1.27 1.27)) hide)
+    )
+    (property "JLCPCB part number" "DNP" (id 4) (at 210.185 23.495 0)
+      (effects (font (size 1.27 1.27)) hide)
+    )
+    (property "LCSC" "DNP" (id 5) (at 210.185 23.495 0)
       (effects (font (size 1.27 1.27)) hide)
     )
@@
       (effects (font (size 1.27 1.27)) (justify left))
     )
-    (property "Value" "0.1uF" (id 1) (at 194.31 86.36 0)
+    (property "Value" "100n" (id 1) (at 194.31 86.36 0)
       (effects (font (size 1.27 1.27)) (justify left))
     )
@@
     )
     (property "Datasheet" "~" (id 3) (at 191.135 85.09 0)
+      (effects (font (size 1.27 1.27)) hide)
+    )
+    (property "JLCPCB part number" "C85866" (id 4) (at 191.135 85.09 0)
+      (effects (font (size 1.27 1.27)) hide)
+    )
+    (property "LCSC" "C85866" (id 5) (at 191.135 85.09 0)
       (effects (font (size 1.27 1.27)) hide)
     )
@@
       (effects (font (size 1.27 1.27)) (justify left))
     )
-    (property "Value" "0.1uF" (id 1) (at 220.98 86.36 0)
+    (property "Value" "100n" (id 1) (at 220.98 86.36 0)
       (effects (font (size 1.27 1.27)) (justify left))
     )
@@
     )
     (property "Datasheet" "~" (id 3) (at 217.805 85.09 0)
+      (effects (font (size 1.27 1.27)) hide)
+    )
+    (property "JLCPCB part number" "C85866" (id 4) (at 217.805 85.09 0)
+      (effects (font (size 1.27 1.27)) hide)
+    )
+    (property "LCSC" "C85866" (id 5) (at 217.805 85.09 0)
       (effects (font (size 1.27 1.27)) hide)
     )
@@
     )
     (path "/24245eb9-ca47-44c8-aef0-c3c799721dfb"
-      (reference "C200") (unit 1) (value "0.33u") (footprint "Capacitor_SMD:CP_Elec_5x5.9")
+      (reference "C200") (unit 1) (value "33u") (footprint "Capacitor_SMD:CP_Elec_5x5.8")
     )
     (path "/eb5e6dc8-0dbf-4532-a1b5-d636bab302c2"
-      (reference "C201") (unit 1) (value "0.1uF") (footprint "Capacitor_SMD:C_0805_2012Metric_Pad1.18x1.45mm_HandSolder")
+      (reference "C201") (unit 1) (value "100n") (footprint "Capacitor_SMD:C_0805_2012Metric_Pad1.18x1.45mm_HandSolder")
     )
     (path "/f65c0be0-dcc8-4944-a91a-8ba24fe6a880"
-      (reference "C202") (unit 1) (value "0.1uF") (footprint "Capacitor_SMD:C_0805_2012Metric_Pad1.18x1.45mm_HandSolder")
+      (reference "C202") (unit 1) (value "100n") (footprint "Capacitor_SMD:C_0805_2012Metric_Pad1.18x1.45mm_HandSolder")
     )
     (path "/a9c1e669-057d-41d2-906c-a906c148ce27/151bf897-7982-4828-a0c7-cdd4ef1dcfcf"
-      (reference "D1") (unit 1) (value "D") (footprint "Diode_SMD:D_0805_2012Metric_Pad1.15x1.40mm_HandSolder")
+      (reference "D1") (unit 1) (value "D") (footprint "Diode_SMD:D_SOD-123F")
     )
     (path "/b0edea89-a55e-4eaf-a3de-ce2754cd615f/e17cf543-52f8-46d4-b1d3-31347d74b5ef"
-      (reference "D21") (unit 1) (value "D") (footprint "Diode_SMD:D_0805_2012Metric_Pad1.15x1.40mm_HandSolder")
+      (reference "D21") (unit 1) (value "D") (footprint "Diode_SMD:D_SOD-123F")
     )
     (path "/e112d131-dec3-432d-a3a2-c0e30c26485b"
@@
     )
     (path "/a9c1e669-057d-41d2-906c-a906c148ce27/8bfe99a0-99b4-4758-a888-a87a75cfcbc2"
-      (reference "R2") (unit 1) (value "R") (footprint "Resistor_SMD:R_1206_3216Metric_Pad1.30x1.75mm_HandSolder")
+      (reference "R2") (unit 1) (value "DNP") (footprint "Resistor_SMD:R_1206_3216Metric_Pad1.30x1.75mm_HandSolder")
     )
     (path "/a9c1e669-057d-41d2-906c-a906c148ce27/042e77e2-61d3-4f4e-a8fa-f65fafcde105"
@@
     )
     (path "/a9c1e669-057d-41d2-906c-a906c148ce27/fb8b83fd-7b28-4035-9d63-2faa45239fe1"
-      (reference "R7") (unit 1) (value "R") (footprint "Resistor_SMD:R_0603_1608Metric_Pad0.98x0.95mm_HandSolder")
+      (reference "R7") (unit 1) (value "100k") (footprint "Resistor_SMD:R_0603_1608Metric_Pad0.98x0.95mm_HandSolder")
     )
     (path "/a9c1e669-057d-41d2-906c-a906c148ce27/efad11de-9fe8-45a7-b373-76b8431e2d5e"
@@
     )
     (path "/a9c1e669-057d-41d2-906c-a906c148ce27/e18ee009-4620-47a5-99a0-796af3c257ef"
-      (reference "R11") (unit 1) (value "R") (footprint "Resistor_SMD:R_0603_1608Metric_Pad0.98x0.95mm_HandSolder")
+      (reference "R11") (unit 1) (value "4.7k") (footprint "Resistor_SMD:R_0603_1608Metric_Pad0.98x0.95mm_HandSolder")
     )
     (path "/a9c1e669-057d-41d2-906c-a906c148ce27/b0ae2d42-278f-4633-b800-509cc4124c4b"
@@
     )
     (path "/b0edea89-a55e-4eaf-a3de-ce2754cd615f/3e7740fe-c488-4c44-9375-364e011d4abc"
-      (reference "R22") (unit 1) (value "R") (footprint "Resistor_SMD:R_1206_3216Metric_Pad1.30x1.75mm_HandSolder")
+      (reference "R22") (unit 1) (value "DNP") (footprint "Resistor_SMD:R_1206_3216Metric_Pad1.30x1.75mm_HandSolder")
     )
     (path "/b0edea89-a55e-4eaf-a3de-ce2754cd615f/6b4a59aa-d044-43c8-8783-3ba72480a6ac"
@@
     )
     (path "/b0edea89-a55e-4eaf-a3de-ce2754cd615f/cb648988-6cef-42c1-9556-bfed799be5e8"
-      (reference "R27") (unit 1) (value "R") (footprint "Resistor_SMD:R_0603_1608Metric_Pad0.98x0.95mm_HandSolder")
+      (reference "R27") (unit 1) (value "100k") (footprint "Resistor_SMD:R_0603_1608Metric_Pad0.98x0.95mm_HandSolder")
     )
     (path "/b0edea89-a55e-4eaf-a3de-ce2754cd615f/d3e8e25d-b131-49d9-b420-528c3245ef60"
@@
     )
     (path "/b0edea89-a55e-4eaf-a3de-ce2754cd615f/35eea9c5-f7e9-4733-ac2c-ecbf80c8f071"
-      (reference "R31") (unit 1) (value "R") (footprint "Resistor_SMD:R_0603_1608Metric_Pad0.98x0.95mm_HandSolder")
+      (reference "R31") (unit 1) (value "4.7k") (footprint "Resistor_SMD:R_0603_1608Metric_Pad0.98x0.95mm_HandSolder")
     )
     (path "/b0edea89-a55e-4eaf-a3de-ce2754cd615f/f3010326-76bc-4e8a-b101-060b583e3d8e"
@@
     )
     (path "/a9c1e669-057d-41d2-906c-a906c148ce27/025c39cd-d314-4dc5-8426-340997e22643"
-      (reference "R200") (unit 1) (value "R") (footprint "Resistor_SMD:R_0603_1608Metric_Pad0.98x0.95mm_HandSolder")
+      (reference "R200") (unit 1) (value "510") (footprint "Resistor_SMD:R_0603_1608Metric_Pad0.98x0.95mm_HandSolder")
     )
     (path "/b0edea89-a55e-4eaf-a3de-ce2754cd615f/768535df-4a17-406e-b978-2f8b1f9c0dd5"
-      (reference "R201") (unit 1) (value "R") (footprint "Resistor_SMD:R_0603_1608Metric_Pad0.98x0.95mm_HandSolder")
+      (reference "R201") (unit 1) (value "150") (footprint "Resistor_SMD:R_0603_1608Metric_Pad0.98x0.95mm_HandSolder")
     )
     (path "/a9c1e669-057d-41d2-906c-a906c148ce27/224206bb-7be7-4fcd-a1c5-b223bf3601b8"
