File: Token_Ring_MAU_Port_1.kicad_sch (KiCad schematic)
At the start: 26 parts, among them J1 RJ45_LED_Shielded_x2, K1 4PDT_relay, Q1 Q_NPN_BEC, Q2 Q_NPN_BEC, T1 Transformer_Token_Ring_1to1_1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, U1 H11A1

Commit message: Add pictures, gerbers, warning note
Parts:
- C1, C2: JLCPCB part number (none) -> C106167; LCSC (none) -> C106167
- C3: JLCPCB part number (none) -> C7225; LCSC (none) -> C7225
- C4, C5: JLCPCB part number (none) -> C282672; LCSC (none) -> C282672
- D1: footprint Diode_SMD:D_0805_2012Metric_Pad1.15x1.40mm_HandSolder -> Diode_SMD:D_SOD-123F; JLCPCB part number (none) -> C108803; LCSC (none) -> C108803
- J1, K1, T1, U1: JLCPCB part number (none) -> DNP; LCSC (none) -> DNP
- Q1, Q2: JLCPCB part number (none) -> C141788; LCSC (none) -> C141788
- R1: JLCPCB part number (none) -> C323071; LCSC (none) -> C323071
- R10: JLCPCB part number (none) -> C403190; LCSC (none) -> C403190
- R11: value R -> 4.7k; JLCPCB part number (none) -> C105428; LCSC (none) -> C105428
- R12, R13, R3, R4: JLCPCB part number (none) -> C21189; LCSC (none) -> C21189
- R2: value R -> DNP; JLCPCB part number (none) -> DNP; LCSC (none) -> DNP
- R200: value R -> 510; JLCPCB part number (none) -> C23193; LCSC (none) -> C23193
- R5, R6: JLCPCB part number (none) -> C445624; LCSC (none) -> C445624
- R7: value R -> 100k; JLCPCB part number (none) -> C150003; LCSC (none) -> C150003
- R8: JLCPCB part number (none) -> C100708; LCSC (none) -> C100708
- R9: JLCPCB part number (none) -> C217936; LCSC (none) -> C217936
