File: Token_Ring_MAU_Port_2.kicad_sch (KiCad schematic)
At the start: 26 parts, among them J1 RJ45_LED_Shielded_x2, K2 4PDT_relay, Q21 Q_NPN_BEC, Q22 Q_NPN_BEC, T2 Transformer_Token_Ring_1to1_1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, U21 H11A1

Commit message: Add pictures, gerbers, warning note
Parts:
- C21, C22: JLCPCB part number (none) -> C106167; LCSC (none) -> C106167
- C23: JLCPCB part number (none) -> C7225; LCSC (none) -> C7225
- C24, C25: JLCPCB part number (none) -> C282672; LCSC (none) -> C282672
- D21: footprint Diode_SMD:D_0805_2012Metric_Pad1.15x1.40mm_HandSolder -> Diode_SMD:D_SOD-123F; JLCPCB part number (none) -> C108803; LCSC (none) -> C108803
- J1, K2, T2, U21: JLCPCB part number (none) -> DNP; LCSC (none) -> DNP
- Q21, Q22: JLCPCB part number (none) -> C141788; LCSC (none) -> C141788
- R201: value R -> 150; JLCPCB part number (none) -> C227596; LCSC (none) -> C227596
- R21: JLCPCB part number (none) -> C323071; LCSC (none) -> C323071
- R22: value R -> DNP; JLCPCB part number (none) -> DNP; LCSC (none) -> DNP
- R23, R24, R32, R33: JLCPCB part number (none) -> C21189; LCSC (none) -> C21189
- R25, R26: JLCPCB part number (none) -> C445624; LCSC (none) -> C445624
- R27: value R -> 100k; JLCPCB part number (none) -> C150003; LCSC (none) -> C150003
- R28: JLCPCB part number (none) -> C100708; LCSC (none) -> C100708
- R29: JLCPCB part number (none) -> C217936; LCSC (none) -> C217936
- R30: JLCPCB part number (none) -> C403190; LCSC (none) -> C403190
- R31: value R -> 4.7k; JLCPCB part number (none) -> C105428; LCSC (none) -> C105428
